File: charger/charger.kicad_sch (KiCad schematic)
At the start: 13 parts, among them J1 USB4515-GF-A_REVA, J2 Screw_Terminal_2_P5.00mm

Commit message: added power/ground planes
Parts:
- renumbered J1 to J2, J2 to J3
Connections:
- net +5V: now also J3.2; no longer J3.1
- net GND: now also J3.1; no longer J3.2
